File: Rx_SelfTest_Module.kicad_sch (KiCad schematic)
At the start: 21 parts, among them J1 SEAM-30-07.0-S-08-1-A-K-TR

Commit message: Ready for production
Parts:
- RF1, RF2, RF3, RF4: value SMA-J-P-H-ST-TH1 -> 132134-15; footprint bynet_SMA:SMA_STR_SAMTEC_SMA-J-P-X-ST-TH1 -> bynet_SMA:SMA_SMD+TH_Amphenol_RF_132134-15; Manufacturer Samtec -> Amphenol RF; mfg P/N SMA-J-P-H-ST-TH1 -> 132134-15
Connections:
- net GNDA: now also RF13.2, RF13.3, RF13.4, RF13.5
Changed lines of the file:
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@@
 	)
 	(junction
+		(at 40.64 57.15)
+		(diameter 0)
+		(color 0 0 0 0)
+	)
+	(junction
 		(at 210.82 101.6)
 		(diameter 0)
@@
 	(wire
 		(pts
-			(xy 40.64 44.45) (xy 40.64 69.85)
+			(xy 40.64 44.45) (xy 40.64 57.15)
 		)
 		(stroke
@@
 	(wire
 		(pts
+			(xy 40.64 57.15) (xy 40.64 69.85)
+		)
+		(stroke
+			(width 0)
+			(type default)
+		)
+	)
+	(wire
+		(pts
 			(xy 88.9 271.78) (xy 88.9 276.86)
 		)
@@
 	(wire
 		(pts
+			(xy 31.75 57.15) (xy 40.64 57.15)
+		)
+		(stroke
+			(width 0)
+			(type default)
+		)
+	)
+	(wire
+		(pts
 			(xy 154.94 118.11) (xy 157.48 118.11)
 		)
@@
 			)
 		)
-		(property "Value" "SMA-J-P-H-ST-TH1"
+		(property "Value" "132134-15"
 			(at 29.0068 268.8336 0)
 			(effects
@@
 			)
 		)
-		(property "Footprint" "bynet_SMA:SMA_STR_SAMTEC_SMA-J-P-X-ST-TH1"
+		(property "Footprint" "bynet_SMA:SMA_SMD+TH_Amphenol_RF_132134-15"
 			(at 29.21 274.32 0)
 			(effects
@@
 			)
 		)
-		(property "Datasheet" "https://www.samtec.com/products/sma-j-p-h-st-th1"
+		(property "Datasheet" "https://www.amphenolrf.com/132134-15.html"
 			(at 29.21 274.32 0)
 			(effects
@@
 			)
 		)
-		(property "mfg P/N" "SMA-J-P-H-ST-TH1"
+		(property "mfg P/N" "132134-15"
 			(at 29.21 274.32 0)
 			(effects
@@
 			)
 		)
-		(property "Manufacturer" "Samtec"
+		(property "Manufacturer" "Amphenol RF"
 			(at 29.21 274.32 0)
 			(effects
@@
 			)
 		)
-		(property "Value" "SMA-J-P-H-ST-TH1"
+		(property "Value" "132134-15"
 			(at 29.0068 207.8736 0)
 			(effects
@@
 			)
 		)
-		(property "Footprint" "bynet_SMA:SMA_STR_SAMTEC_SMA-J-P-X-ST-TH1"
+		(property "Footprint" "bynet_SMA:SMA_SMD+TH_Amphenol_RF_132134-15"
 			(at 29.21 213.36 0)
 			(effects
@@
 			)
 		)
-		(property "Datasheet" "https://www.samtec.com/products/sma-j-p-h-st-th1"
+		(property "Datasheet" "https://www.amphenolrf.com/132134-15.html"
 			(at 29.21 213.36 0)
 			(effects
@@
 			)
 		)
-		(property "mfg P/N" "SMA-J-P-H-ST-TH1"
+		(property "mfg P/N" "132134-15"
 			(at 29.21 213.36 0)
 			(effects
@@
 			)
 		)
-		(property "Manufacturer" "Samtec"
+		(property "Manufacturer" "Amphenol RF"
 			(at 29.21 213.36 0)
 			(effects
@@
 			)
 		)
-		(property "Value" "SMA-J-P-H-ST-TH1"
+		(property "Value" "132134-15"
 			(at 29.0068 248.5136 0)
 			(effects
@@
 			)
 		)
-		(property "Footprint" "bynet_SMA:SMA_STR_SAMTEC_SMA-J-P-X-ST-TH1"
+		(property "Footprint" "bynet_SMA:SMA_SMD+TH_Amphenol_RF_132134-15"
 			(at 29.21 254 0)
 			(effects
@@
 			)
 		)
-		(property "Datasheet" "https://www.samtec.com/products/sma-j-p-h-st-th1"
+		(property "Datasheet" "https://www.amphenolrf.com/132134-15.html"
 			(at 29.21 254 0)
 			(effects
@@
 			)
 		)
-		(property "mfg P/N" "SMA-J-P-H-ST-TH1"
+		(property "mfg P/N" "132134-15"
 			(at 29.21 254 0)
 			(effects
@@
 			)
 		)
-		(property "Manufacturer" "Samtec"
+		(property "Manufacturer" "Amphenol RF"
 			(at 29.21 254 0)
 			(effects
@@
 			)
 		)
-		(property "Value" "SMA-J-P-H-ST-TH1"
+		(property "Value" "132134-15"
 			(at 29.0068 226.9236 0)
 			(effects
@@
 			)
 		)
-		(property "Footprint" "bynet_SMA:SMA_STR_SAMTEC_SMA-J-P-X-ST-TH1"
+		(property "Footprint" "bynet_SMA:SMA_SMD+TH_Amphenol_RF_132134-15"
 			(at 29.21 232.41 0)
 			(effects
@@
 			)
 		)
-		(property "Datasheet" "https://www.samtec.com/products/sma-j-p-h-st-th1"
+		(property "Datasheet" "https://www.amphenolrf.com/132134-15.html"
 			(at 29.21 232.41 0)
 			(effects
@@
 			)
 		)
-		(property "mfg P/N" "SMA-J-P-H-ST-TH1"
+		(property "mfg P/N" "132134-15"
 			(at 29.21 232.41 0)
 			(effects
@@
 			)
 		)
-		(property "Manufacturer" "Samtec"
+		(property "Manufacturer" "Amphenol RF"
 			(at 29.21 232.41 0)
 			(effects
